Commit message: Fixed bug in pioneer 3dx gazebo model that made it turn the wrong way Added sound alert to estop Removed unused parameter from gazebo launch file

File: src/pioneer_hallway/config/urdf/pioneer3dx.xacro (robot description, xacro)
@@ -163,5 +163,5 @@
   	<joint_properties damping="0.0" friction="0.0" />-->
 		<parent link="base_link"/>
-		<child link="left_wheel"/>
+		<child link="right_wheel"/>
 	</joint>
 	<link name="left_wheel">
@@ -215,5 +215,5 @@
   	<joint_properties damping="0.0" friction="0.0" />-->
 		<parent link="base_link"/>
-		<child link="right_wheel"/>
+		<child link="left_wheel"/>
 	</joint>
 	<link name="right_wheel">

Commit message: Added an rviz configuration file that will be used only in simulation Minor modifications to the rviz file used in real life Modified the gazebo an xacro files of the p3dx model to add the sonars Increased amcl's sampling frequency in both amcl launch files Added configuration parameters to simulation and real life launch files Minor modifications to rviz launchfile so it can use different configuration files Added the sonar transfor to the tf broadcaster

File: src/pioneer_hallway/config/urdf/pioneer3dx.xacro (robot description, xacro)
@@ -268,5 +268,5 @@
 		</inertial>
 		<visual name="base_visual">
-			<origin xyz="0 0 0" rpy="0 0 0"/>
+			<origin xyz="0 0 0" rpy="0 0 -3.14159"/>
 			<geometry name="pioneer_geom">
 				<mesh filename="package://pioneer_description/meshes/p3dx_meshes/front_sonar.stl"/>
@@ -282,5 +282,5 @@
 	</link>
 	<joint name="base_front_joint" type="fixed">
-		<origin xyz="-0.198 0 0.208" rpy="0 0 0"/>
+		<origin xyz="-0.198 0 0.208" rpy="0 0 -3.14159"/>
 		<parent link="base_link"/>
 		<child link="front_sonar"/>

Commit message: Modified the p3dx gazebo model to increase its weight and set a maximum acceleration Deleted unused wav file Updated estop to use the current speed and maximum deceleration to predict collisions Updated rosaria launch file to set the robot's maximum acceleration to 0.6 m/s Updated teleop node to allow easier testing

File: src/pioneer_hallway/config/urdf/pioneer3dx.xacro (robot description, xacro)
@@ -30,5 +30,5 @@
 		</collision>
 		<inertial>
-		  <mass value="5.67"/>
+		  <mass value="25"/>
 		  <inertia ixx="0.07" ixy="0" ixz="0"
 		    iyy="0.08" iyz="0"
